File: Soraduino/soraduino.brd (EAGLE design)
At the start: 87.3 x 81.3 mm, 23 parts, among them IC1 ATMEGA168-AU, IC2 317EMP, IC3 317EMP

Commit message: GPS、Digital出力を一旦削除
Parts:
- removed DIGITAL: (no value), pinhead:1X06
- removed GPS-SUP: (no value), con-lstb:MA04-2
Connections:
- removed net N$36: GPS-SUP.8, IC1.32
- removed net N$37: GPS-SUP.6, IC1.2
- removed net N$39: DIGITAL.1, IC1.9
- removed net N$40: DIGITAL.2, IC1.10
- removed net N$41: DIGITAL.3, IC1.11
- removed net N$42: DIGITAL.4, IC1.12
- removed net N$47: DIGITAL.5, IC1.16
- net GND: no longer GPS-SUP.3, GPS-SUP.4, GPS-SUP.5
- net N$6: no longer GPS-SUP.1
- net N$7: no longer GPS-SUP.2, GPS-SUP.7
Changed lines of the file:
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@@
 <element name="R1" library="rcl" package="R0603" value="1k" x="36.83" y="81.28" rot="MR180"/>
 <element name="R2" library="rcl" package="R0603" value="1k" x="38.1" y="36.83" rot="MR0"/>
-<element name="DIGITAL" library="pinhead" package="1X06" value="" x="21.59" y="58.42"/>
 <element name="SV1" library="con-lstb" package="MA20-2" value="" x="88.9" y="53.34" rot="MR90">
 <attribute name="OC_NEWARK" value="unknown" x="88.9" y="53.34" size="1.778" layer="28" rot="MR90" display="off"/>
@@
 <attribute name="OC_FARNELL" value="unknown" x="62.23" y="59.69" size="1.778" layer="28" rot="MR270" display="off"/>
 </element>
-<element name="GPS-SUP" library="con-lstb" package="MA04-2" value="" x="53.34" y="59.69" rot="MR270">
-<attribute name="OC_NEWARK" value="unknown" x="53.34" y="59.69" size="1.778" layer="28" rot="MR270" display="off"/>
-<attribute name="MPN" value="" x="53.34" y="59.69" size="1.778" layer="28" rot="MR270" display="off"/>
-<attribute name="MF" value="" x="53.34" y="59.69" size="1.778" layer="28" rot="MR270" display="off"/>
-<attribute name="OC_FARNELL" value="unknown" x="53.34" y="59.69" size="1.778" layer="28" rot="MR270" display="off"/>
-</element>
 </elements>
 <signals>
@@
 <contactref element="C4" pad="2"/>
 <contactref element="I2C-ACC" pad="2"/>
-<contactref element="GPS-SUP" pad="1"/>
 <contactref element="I2C-ACC" pad="1"/>
 <wire x1="39.1" y1="40.64" x2="39.1" y2="50.089" width="0.254" layer="16"/>
 <wire x1="39.1" y1="50.089" x2="35.56" y2="50.089" width="0.254" layer="16"/>
 <wire x1="60.96" y1="63.5" x2="63.5" y2="63.5" width="0" layer="19" extent="1-1"/>
-<wire x1="54.61" y1="63.5" x2="60.96" y2="63.5" width="0" layer="19" extent="1-1"/>
-<wire x1="39.1" y1="50.089" x2="54.61" y2="63.5" width="0" layer="19" extent="16-16"/>
+<wire x1="39.1" y1="50.089" x2="60.96" y2="63.5" width="0" layer="19" extent="16-16"/>
 <wire x1="41.07" y1="38.21" x2="39.1" y2="40.64" width="0" layer="19" extent="16-16"/>
 </signal>
@@
 <wire x1="42.3926" y1="70.58" x2="60.96" y2="68.58" width="0" layer="19" extent="1-1"/>
 </signal>
-<signal name="N$36">
-<contactref element="IC1" pad="32"/>
-<contactref element="GPS-SUP" pad="8"/>
-<wire x1="35.3" y1="72.8726" x2="52.07" y2="55.88" width="0" layer="19" extent="1-1"/>
-</signal>
-<signal name="N$37">
-<contactref element="IC1" pad="2"/>
-<contactref element="GPS-SUP" pad="6"/>
-<wire x1="33.8074" y1="70.58" x2="52.07" y2="58.42" width="0" layer="19" extent="1-1"/>
-</signal>
 <signal name="N$38">
 <contactref element="IC4" pad="27"/>
 <contactref element="R2" pad="1"/>
 <wire x1="38.95" y1="36.83" x2="73.895" y2="49.17" width="0" layer="19" extent="16-16"/>
-</signal>
-<signal name="N$39">
-<contactref element="IC1" pad="9"/>
-<contactref element="DIGITAL" pad="1"/>
-<wire x1="15.24" y1="58.42" x2="35.3" y2="64.2874" width="0" layer="19" extent="1-1"/>
-</signal>
-<signal name="N$40">
-<contactref element="IC1" pad="10"/>
-<contactref element="DIGITAL" pad="2"/>
-<wire x1="17.78" y1="58.42" x2="36.1" y2="64.2874" width="0" layer="19" extent="1-1"/>
-</signal>
-<signal name="N$41">
-<contactref element="IC1" pad="11"/>
-<contactref element="DIGITAL" pad="3"/>
-<wire x1="20.32" y1="58.42" x2="36.9" y2="64.2874" width="0" layer="19" extent="1-1"/>
-</signal>
-<signal name="N$42">
-<contactref element="IC1" pad="12"/>
-<contactref element="DIGITAL" pad="4"/>
-<wire x1="22.86" y1="58.42" x2="37.7" y2="64.2874" width="0" layer="19" extent="1-1"/>
-</signal>
-<signal name="N$47">
-<contactref element="IC1" pad="16"/>
-<contactref element="DIGITAL" pad="5"/>
-<wire x1="25.4" y1="58.42" x2="40.9" y2="64.2874" width="0" layer="19" extent="1-1"/>
 </signal>
 <signal name="N$9">
@@
 </signal>
 <signal name="N$7">
-<contactref element="GPS-SUP" pad="7"/>
 <contactref element="IC3" pad="4"/>
 <contactref element="C6" pad="2"/>
@@
 <contactref element="IC4" pad="26"/>
 <contactref element="JAIRO-ANA" pad="2"/>
-<contactref element="GPS-SUP" pad="2"/>
 <wire x1="28.94" y1="40.64" x2="28.94" y2="50.089" width="0.254" layer="16"/>
 <wire x1="28.94" y1="50.089" x2="25.4" y2="50.089" width="0.254" layer="16"/>
 <wire x1="28.94" y1="40.64" x2="28.94" y2="43.45" width="0.254" layer="16"/>
 <wire x1="28.94" y1="43.45" x2="30.48" y2="43.45" width="0.254" layer="16"/>
-<wire x1="52.07" y1="63.5" x2="60.96" y2="76.2" width="0" layer="19" extent="1-1"/>
-<wire x1="54.61" y1="55.88" x2="52.07" y2="63.5" width="0" layer="19" extent="1-1"/>
-<wire x1="42.3926" y1="66.58" x2="52.07" y2="63.5" width="0" layer="19" extent="1-1"/>
+<wire x1="42.3926" y1="66.58" x2="60.96" y2="76.2" width="0" layer="19" extent="1-1"/>
 <wire x1="33.8074" y1="67.38" x2="42.3926" y2="66.58" width="0" layer="19" extent="1-1"/>
 <wire x1="33.8074" y1="68.98" x2="33.8074" y2="67.38" width="0" layer="19" extent="1-1"/>
 <wire x1="35.98" y1="81.28" x2="33.8074" y2="68.98" width="0" layer="19" extent="1-16"/>
 <wire x1="28.94" y1="50.089" x2="33.8074" y2="67.38" width="0" layer="19" extent="1-16"/>
-<wire x1="73.075" y1="49.62" x2="54.61" y2="55.88" width="0" layer="19" extent="16-16"/>
+<wire x1="30.48" y1="19.05" x2="28.94" y2="40.64" width="0" layer="19" extent="16-16"/>
+<wire x1="73.075" y1="49.62" x2="60.96" y2="76.2" width="0" layer="19" extent="16-16"/>
 <wire x1="74.545" y1="49.17" x2="73.075" y2="49.62" width="0" layer="19" extent="16-16"/>
-<wire x1="30.48" y1="19.05" x2="28.94" y2="40.64" width="0" layer="19" extent="16-16"/>
 </signal>
 <signal name="N$25">
@@
 </signal>
 <signal name="GND">
-<contactref element="GPS-SUP" pad="4"/>
 <contactref element="C1" pad="1"/>
 <contactref element="C2" pad="1"/>
@@
 <contactref element="SV2" pad="1"/>
 <contactref element="JAIRO-ANA" pad="4"/>
-<contactref element="GPS-SUP" pad="3"/>
-<contactref element="GPS-SUP" pad="5"/>
 <contactref element="I2C-ACC" pad="3"/>
 <contactref element="I2C-ACC" pad="4"/>
@@
 <wire x1="92.71" y1="67.31" x2="92.71" y2="59.69" width="0.254" layer="16"/>
 <wire x1="92.71" y1="69.85" x2="92.71" y2="72.39" width="0.254" layer="16"/>
+<wire x1="73.075" y1="54.52" x2="73.075" y2="52.07" width="0.254" layer="16"/>
+<wire x1="73.075" y1="52.07" x2="74.93" y2="52.07" width="0.254" layer="16"/>
 <wire x1="60.96" y1="60.96" x2="60.96" y2="73.66" width="0" layer="19" extent="1-1"/>
 <wire x1="63.5" y1="60.96" x2="60.96" y2="60.96" width="0" layer="19" extent="1-1"/>
-<wire x1="54.61" y1="60.96" x2="60.96" y2="60.96" width="0" layer="19" extent="1-1"/>
-<wire x1="52.07" y1="60.96" x2="54.61" y2="60.96" width="0" layer="19" extent="1-1"/>
-<wire x1="54.61" y1="58.42" x2="54.61" y2="60.96" width="0" layer="19" extent="1-1"/>
-<wire x1="76.495" y1="54.97" x2="73.075" y2="54.52" width="0" layer="19" extent="16-16"/>
-<wire x1="77.47" y1="52.07" x2="76.495" y2="54.97" width="0" layer="19" extent="16-16"/>
-<wire x1="42.3926" y1="68.98" x2="52.07" y2="60.96" width="0" layer="19" extent="1-1"/>
+<wire x1="73.075" y1="54.52" x2="63.5" y2="60.96" width="0" layer="19" extent="16-16"/>
+<wire x1="76.495" y1="54.97" x2="74.93" y2="52.07" width="0" layer="19" extent="16-16"/>
+<wire x1="92.71" y1="54.61" x2="76.495" y2="54.97" width="0" layer="19" extent="16-16"/>
+<wire x1="42.3926" y1="68.98" x2="60.96" y2="73.66" width="0" layer="19" extent="1-1"/>
 <wire x1="33.8074" y1="69.78" x2="42.3926" y2="68.98" width="0" layer="19" extent="1-1"/>
 <wire x1="33.8074" y1="68.18" x2="33.8074" y2="69.78" width="0" layer="19" extent="1-1"/>
 <wire x1="20.32" y1="69.85" x2="33.8074" y2="69.78" width="0" layer="19" extent="1-1"/>
 <wire x1="20.32" y1="72.39" x2="20.32" y2="69.85" width="0" layer="19" extent="1-1"/>
-<wire x1="92.71" y1="52.07" x2="77.47" y2="52.07" width="0" layer="19" extent="16-16"/>
 <wire x1="30.48" y1="52.07" x2="33.8074" y2="68.18" width="0" layer="19" extent="1-16"/>
 <wire x1="41.07" y1="20.21" x2="37.25" y2="36.83" width="0" layer="19" extent="16-16"/>
 <wire x1="35.56" y1="19.05" x2="41.07" y2="20.21" width="0" layer="19" extent="1-1"/>
-<wire x1="73.075" y1="54.52" x2="73.075" y2="52.07" width="0.254" layer="16"/>
-<wire x1="73.075" y1="52.07" x2="74.93" y2="52.07" width="0.254" layer="16"/>
-<wire x1="74.93" y1="52.07" x2="76.495" y2="54.97" width="0" layer="19" extent="1-16"/>
 </signal>
 <signal name="VCC">
