File: Soraduino/soraduino.brd (EAGLE design)
At the start: 87.3 x 81.3 mm, 21 parts, among them IC1 ATMEGA168-AU, IC2 317EMP, IC3 317EMP

Commit message: 仮配線完了
Parts:
- moved USB 81.1 mm to (81.3, 81.3)
- moved C2 46.2 mm to (67.3, 57.1)
- moved C1 44.5 mm to (67.3, 73.7)
- moved XB1 42.6 mm to (71.1, 67.3)
- moved R2 41.0 mm to (78.7, 41.9)
- moved JAIRO-ANA 39.7 mm to (67.3, 33.0)
- moved C5 37.4 mm to (67.3, 50.8), turned to 270 degrees
- moved C8 37.4 mm to (77.5, 74.9), turned to 90 degrees
- moved R1 37.4 mm to (73.7, 74.9), turned to 270 degrees
- moved IC2 37.2 mm to (72.4, 52.1)
- moved IC3 37.2 mm to (62.2, 52.1)
- moved IC1 37.0 mm to (74.9, 64.8), flipped to the bottom, turned to 135 degrees
- moved Q1 37.0 mm to (66.0, 64.8)
- moved C6 37.0 mm to (64.8, 44.5)
- moved C7 37.0 mm to (61.0, 44.5)
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Routing:
- net N$31: track 0.00 -> 107.1 mm, vias 0 -> 2
- net N$35: track 0.00 -> 96.5 mm, vias 0 -> 6
- net N$45: track 0.00 -> 86.2 mm, vias 0 -> 2
- net GND: track 127.7 -> 211.1 mm, vias 0 -> 4
- net N$44: track 0.00 -> 80.6 mm, vias 0 -> 7
- net N$26: track 0.00 -> 80.3 mm, vias 0 -> 6
- net N$28: track 0.00 -> 79.4 mm, vias 0 -> 2
- net N$7: track 17.3 -> 93.9 mm, vias 0 -> 3
- net N$8: track 31.1 -> 107.4 mm, vias 0 -> 4
- net N$6: track 13.0 -> 78.0 mm, vias 0 -> 2
- net N$12: track 26.0 -> 87.5 mm, vias 0 -> 2
- net N$3: track 0.00 -> 60.5 mm, vias 0 -> 2
- net N$22: track 24.1 -> 76.4 mm, vias 0 -> 4
- net N$30: track 0.00 -> 51.6 mm, vias 0 -> 4
- net N$25: track 0.00 -> 49.8 mm, vias 0 -> 1
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Other:
- board size 87.3 x 81.3 mm -> 42.9 x 59.7 mm

Commit message: back GPS 1
Parts:
- moved USB 81.1 mm to (29.2, 19.1)
- moved C2 46.2 mm to (22.9, 69.8)
- moved C1 44.5 mm to (22.9, 72.4)
- moved XB1 42.6 mm to (52.1, 29.2)
- moved R2 41.0 mm to (38.1, 36.8)
- moved JAIRO-ANA 39.7 mm to (62.2, 72.4)
- moved C5 37.4 mm to (30.5, 44.5), turned to 90 degrees
- moved C8 37.4 mm to (40.6, 81.3), turned to 180 degrees
- moved R1 37.4 mm to (36.8, 81.3), turned to 180 degrees
- moved IC2 37.2 mm to (35.6, 47.0)
- moved IC3 37.2 mm to (25.4, 47.0)
- moved IC1 37.0 mm to (38.1, 68.6), flipped to the top, turned to 0 degrees
- moved Q1 37.0 mm to (29.2, 68.6)
- moved C6 37.0 mm to (27.9, 40.6)
- moved C7 37.0 mm to (24.1, 40.6)
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Routing:
- net N$31: track 107.1 -> 0.00 mm, vias 2 -> 0
- net N$35: track 96.5 -> 0.00 mm, vias 6 -> 0
- net N$45: track 86.2 -> 0.00 mm, vias 2 -> 0
- net GND: track 211.1 -> 127.7 mm, vias 4 -> 0
- net N$44: track 80.6 -> 0.00 mm, vias 7 -> 0
- net N$26: track 80.3 -> 0.00 mm, vias 6 -> 0
- net N$28: track 79.4 -> 0.00 mm, vias 2 -> 0
- net N$7: track 93.9 -> 17.3 mm, vias 3 -> 0
- net N$8: track 107.4 -> 31.1 mm, vias 4 -> 0
- net N$6: track 78.0 -> 13.0 mm, vias 2 -> 0
- net N$12: track 87.5 -> 26.0 mm, vias 2 -> 0
- net N$3: track 60.5 -> 0.00 mm, vias 2 -> 0
- net N$22: track 76.4 -> 24.1 mm, vias 4 -> 0
- net N$30: track 51.6 -> 0.00 mm, vias 4 -> 0
- net N$25: track 49.8 -> 0.00 mm, vias 1 -> 0
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Other:
- board size 42.9 x 59.7 mm -> 87.3 x 81.3 mm

Commit message: Revert "GPS、Digital出力を一旦削除"
This reverts commit f31cc228a309c3dd5619f128104a36497abb7aed.
Parts:
- added DIGITAL: (no value), pinhead:1X06
- added GPS-SUP: (no value), con-lstb:MA04-2
Connections:
- new net N$36: GPS-SUP.8, IC1.32
- new net N$37: GPS-SUP.6, IC1.2
- new net N$39: DIGITAL.1, IC1.9
- new net N$40: DIGITAL.2, IC1.10
- new net N$41: DIGITAL.3, IC1.11
- new net N$42: DIGITAL.4, IC1.12
- new net N$47: DIGITAL.5, IC1.16
- net GND: now also GPS-SUP.3, GPS-SUP.4, GPS-SUP.5
- net N$6: now also GPS-SUP.1
- net N$7: now also GPS-SUP.2, GPS-SUP.7
Changed lines of the file:
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@@
 <element name="R1" library="rcl" package="R0603" value="1k" x="36.83" y="81.28" rot="MR180"/>
 <element name="R2" library="rcl" package="R0603" value="1k" x="38.1" y="36.83" rot="MR0"/>
+<element name="DIGITAL" library="pinhead" package="1X06" value="" x="21.59" y="58.42"/>
 <element name="SV1" library="con-lstb" package="MA20-2" value="" x="88.9" y="53.34" rot="MR90">
 <attribute name="OC_NEWARK" value="unknown" x="88.9" y="53.34" size="1.778" layer="28" rot="MR90" display="off"/>
@@
 <attribute name="OC_FARNELL" value="unknown" x="62.23" y="59.69" size="1.778" layer="28" rot="MR270" display="off"/>
 </element>
+<element name="GPS-SUP" library="con-lstb" package="MA04-2" value="" x="53.34" y="59.69" rot="MR270">
+<attribute name="OC_NEWARK" value="unknown" x="53.34" y="59.69" size="1.778" layer="28" rot="MR270" display="off"/>
+<attribute name="MPN" value="" x="53.34" y="59.69" size="1.778" layer="28" rot="MR270" display="off"/>
+<attribute name="MF" value="" x="53.34" y="59.69" size="1.778" layer="28" rot="MR270" display="off"/>
+<attribute name="OC_FARNELL" value="unknown" x="53.34" y="59.69" size="1.778" layer="28" rot="MR270" display="off"/>
+</element>
 </elements>
 <signals>
@@
 <contactref element="C4" pad="2"/>
 <contactref element="I2C-ACC" pad="2"/>
+<contactref element="GPS-SUP" pad="1"/>
 <contactref element="I2C-ACC" pad="1"/>
 <wire x1="39.1" y1="40.64" x2="39.1" y2="50.089" width="0.254" layer="16"/>
 <wire x1="39.1" y1="50.089" x2="35.56" y2="50.089" width="0.254" layer="16"/>
 <wire x1="60.96" y1="63.5" x2="63.5" y2="63.5" width="0" layer="19" extent="1-1"/>
-<wire x1="39.1" y1="50.089" x2="60.96" y2="63.5" width="0" layer="19" extent="16-16"/>
+<wire x1="54.61" y1="63.5" x2="60.96" y2="63.5" width="0" layer="19" extent="1-1"/>
+<wire x1="39.1" y1="50.089" x2="54.61" y2="63.5" width="0" layer="19" extent="16-16"/>
 <wire x1="41.07" y1="38.21" x2="39.1" y2="40.64" width="0" layer="19" extent="16-16"/>
 </signal>
@@
 <wire x1="42.3926" y1="70.58" x2="60.96" y2="68.58" width="0" layer="19" extent="1-1"/>
 </signal>
+<signal name="N$36">
+<contactref element="IC1" pad="32"/>
+<contactref element="GPS-SUP" pad="8"/>
+<wire x1="35.3" y1="72.8726" x2="52.07" y2="55.88" width="0" layer="19" extent="1-1"/>
+</signal>
+<signal name="N$37">
+<contactref element="IC1" pad="2"/>
+<contactref element="GPS-SUP" pad="6"/>
+<wire x1="33.8074" y1="70.58" x2="52.07" y2="58.42" width="0" layer="19" extent="1-1"/>
+</signal>
 <signal name="N$38">
 <contactref element="IC4" pad="27"/>
 <contactref element="R2" pad="1"/>
 <wire x1="38.95" y1="36.83" x2="73.895" y2="49.17" width="0" layer="19" extent="16-16"/>
+</signal>
+<signal name="N$39">
+<contactref element="IC1" pad="9"/>
+<contactref element="DIGITAL" pad="1"/>
+<wire x1="15.24" y1="58.42" x2="35.3" y2="64.2874" width="0" layer="19" extent="1-1"/>
+</signal>
+<signal name="N$40">
+<contactref element="IC1" pad="10"/>
+<contactref element="DIGITAL" pad="2"/>
+<wire x1="17.78" y1="58.42" x2="36.1" y2="64.2874" width="0" layer="19" extent="1-1"/>
+</signal>
+<signal name="N$41">
+<contactref element="IC1" pad="11"/>
+<contactref element="DIGITAL" pad="3"/>
+<wire x1="20.32" y1="58.42" x2="36.9" y2="64.2874" width="0" layer="19" extent="1-1"/>
+</signal>
+<signal name="N$42">
+<contactref element="IC1" pad="12"/>
+<contactref element="DIGITAL" pad="4"/>
+<wire x1="22.86" y1="58.42" x2="37.7" y2="64.2874" width="0" layer="19" extent="1-1"/>
+</signal>
+<signal name="N$47">
+<contactref element="IC1" pad="16"/>
+<contactref element="DIGITAL" pad="5"/>
+<wire x1="25.4" y1="58.42" x2="40.9" y2="64.2874" width="0" layer="19" extent="1-1"/>
 </signal>
 <signal name="N$9">
@@
 </signal>
 <signal name="N$7">
+<contactref element="GPS-SUP" pad="7"/>
 <contactref element="IC3" pad="4"/>
 <contactref element="C6" pad="2"/>
@@
 <contactref element="IC4" pad="26"/>
 <contactref element="JAIRO-ANA" pad="2"/>
+<contactref element="GPS-SUP" pad="2"/>
 <wire x1="28.94" y1="40.64" x2="28.94" y2="50.089" width="0.254" layer="16"/>
 <wire x1="28.94" y1="50.089" x2="25.4" y2="50.089" width="0.254" layer="16"/>
 <wire x1="28.94" y1="40.64" x2="28.94" y2="43.45" width="0.254" layer="16"/>
 <wire x1="28.94" y1="43.45" x2="30.48" y2="43.45" width="0.254" layer="16"/>
-<wire x1="42.3926" y1="66.58" x2="60.96" y2="76.2" width="0" layer="19" extent="1-1"/>
+<wire x1="52.07" y1="63.5" x2="60.96" y2="76.2" width="0" layer="19" extent="1-1"/>
+<wire x1="54.61" y1="55.88" x2="52.07" y2="63.5" width="0" layer="19" extent="1-1"/>
+<wire x1="42.3926" y1="66.58" x2="52.07" y2="63.5" width="0" layer="19" extent="1-1"/>
 <wire x1="33.8074" y1="67.38" x2="42.3926" y2="66.58" width="0" layer="19" extent="1-1"/>
 <wire x1="33.8074" y1="68.98" x2="33.8074" y2="67.38" width="0" layer="19" extent="1-1"/>
 <wire x1="35.98" y1="81.28" x2="33.8074" y2="68.98" width="0" layer="19" extent="1-16"/>
 <wire x1="28.94" y1="50.089" x2="33.8074" y2="67.38" width="0" layer="19" extent="1-16"/>
+<wire x1="73.075" y1="49.62" x2="54.61" y2="55.88" width="0" layer="19" extent="16-16"/>
+<wire x1="74.545" y1="49.17" x2="73.075" y2="49.62" width="0" layer="19" extent="16-16"/>
 <wire x1="30.48" y1="19.05" x2="28.94" y2="40.64" width="0" layer="19" extent="16-16"/>
-<wire x1="73.075" y1="49.62" x2="60.96" y2="76.2" width="0" layer="19" extent="16-16"/>
-<wire x1="74.545" y1="49.17" x2="73.075" y2="49.62" width="0" layer="19" extent="16-16"/>
 </signal>
 <signal name="N$25">
@@
 </signal>
 <signal name="GND">
+<contactref element="GPS-SUP" pad="4"/>
 <contactref element="C1" pad="1"/>
 <contactref element="C2" pad="1"/>
@@
 <contactref element="SV2" pad="1"/>
 <contactref element="JAIRO-ANA" pad="4"/>
+<contactref element="GPS-SUP" pad="3"/>
+<contactref element="GPS-SUP" pad="5"/>
 <contactref element="I2C-ACC" pad="3"/>
 <contactref element="I2C-ACC" pad="4"/>
@@
 <wire x1="92.71" y1="67.31" x2="92.71" y2="59.69" width="0.254" layer="16"/>
 <wire x1="92.71" y1="69.85" x2="92.71" y2="72.39" width="0.254" layer="16"/>
-<wire x1="73.075" y1="54.52" x2="73.075" y2="52.07" width="0.254" layer="16"/>
-<wire x1="73.075" y1="52.07" x2="74.93" y2="52.07" width="0.254" layer="16"/>
 <wire x1="60.96" y1="60.96" x2="60.96" y2="73.66" width="0" layer="19" extent="1-1"/>
 <wire x1="63.5" y1="60.96" x2="60.96" y2="60.96" width="0" layer="19" extent="1-1"/>
-<wire x1="73.075" y1="54.52" x2="63.5" y2="60.96" width="0" layer="19" extent="16-16"/>
-<wire x1="76.495" y1="54.97" x2="74.93" y2="52.07" width="0" layer="19" extent="16-16"/>
-<wire x1="92.71" y1="54.61" x2="76.495" y2="54.97" width="0" layer="19" extent="16-16"/>
-<wire x1="42.3926" y1="68.98" x2="60.96" y2="73.66" width="0" layer="19" extent="1-1"/>
+<wire x1="54.61" y1="60.96" x2="60.96" y2="60.96" width="0" layer="19" extent="1-1"/>
+<wire x1="52.07" y1="60.96" x2="54.61" y2="60.96" width="0" layer="19" extent="1-1"/>
+<wire x1="54.61" y1="58.42" x2="54.61" y2="60.96" width="0" layer="19" extent="1-1"/>
+<wire x1="76.495" y1="54.97" x2="73.075" y2="54.52" width="0" layer="19" extent="16-16"/>
+<wire x1="77.47" y1="52.07" x2="76.495" y2="54.97" width="0" layer="19" extent="16-16"/>
+<wire x1="42.3926" y1="68.98" x2="52.07" y2="60.96" width="0" layer="19" extent="1-1"/>
 <wire x1="33.8074" y1="69.78" x2="42.3926" y2="68.98" width="0" layer="19" extent="1-1"/>
 <wire x1="33.8074" y1="68.18" x2="33.8074" y2="69.78" width="0" layer="19" extent="1-1"/>
 <wire x1="20.32" y1="69.85" x2="33.8074" y2="69.78" width="0" layer="19" extent="1-1"/>
 <wire x1="20.32" y1="72.39" x2="20.32" y2="69.85" width="0" layer="19" extent="1-1"/>
+<wire x1="92.71" y1="52.07" x2="77.47" y2="52.07" width="0" layer="19" extent="16-16"/>
 <wire x1="30.48" y1="52.07" x2="33.8074" y2="68.18" width="0" layer="19" extent="1-16"/>
 <wire x1="41.07" y1="20.21" x2="37.25" y2="36.83" width="0" layer="19" extent="16-16"/>
 <wire x1="35.56" y1="19.05" x2="41.07" y2="20.21" width="0" layer="19" extent="1-1"/>
+<wire x1="73.075" y1="54.52" x2="73.075" y2="52.07" width="0.254" layer="16"/>
+<wire x1="73.075" y1="52.07" x2="74.93" y2="52.07" width="0.254" layer="16"/>
+<wire x1="74.93" y1="52.07" x2="76.495" y2="54.97" width="0" layer="19" extent="1-16"/>
 </signal>
 <signal name="VCC">

Commit message: 回路をとりあえず完成
Parts:
- added R3, R4, R5: 1k, rcl:R0603
- added RED, YEL1, YEL2: (no value), led:CHIPLED_1206
- moved USB 88.0 mm to (91.4, 81.3)
- moved C2 61.4 mm to (83.8, 77.5)
- moved C1 58.4 mm to (81.3, 73.7)
- moved C3 57.1 mm to (91.4, 40.6), flipped to the top
- moved Q1 54.7 mm to (83.8, 66.0)
- moved IC2 53.3 mm to (88.9, 47.0), flipped to the top
- moved C7 49.5 mm to (73.7, 40.6), flipped to the top
- moved C5 48.3 mm to (78.7, 43.2), flipped to the top
- moved C4 48.3 mm to (86.4, 40.6), flipped to the top, turned to 0 degrees
- moved IC3 45.7 mm to (71.1, 47.0), flipped to the top
- moved GPS-SUP 45.2 mm to (88.9, 31.8)
- moved R2 44.9 mm to (82.5, 43.2), flipped to the top, turned to 270 degrees
- moved DIGITAL 43.4 mm to (62.2, 43.2), turned to 270 degrees
- moved XB1 41.9 mm to (76.2, 63.5)
- moved JAIRO-ANA 41.3 mm to (69.8, 31.8)
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Connections:
- new net N$10: R3.2, RED.A
- new net N$46: R4.2, YEL1.A
- new net N$48: R5.2, YEL2.A
- net GND: now also RED.C, YEL1.C, YEL2.C
- net N$39: now also R4.1
- net N$40: now also R5.1
- net VCC: now also R3.1
Routing:
- net GND: track 127.7 -> 290.3 mm, vias 0 -> 5
- net N$7: track 17.3 -> 167.5 mm, vias 0 -> 5
- net N$43: track 0.00 -> 125.0 mm, vias 0 -> 2
- net N$32: track 0.00 -> 124.3 mm, vias 0 -> 2
- net N$37: track 0.00 -> 108.9 mm
- net N$25: track 0.00 -> 106.6 mm, vias 0 -> 2
- net N$6: track 13.0 -> 113.3 mm, vias 0 -> 5
- net N$16: track 10.9 -> 99.2 mm, vias 0 -> 1
- net N$31: track 0.00 -> 85.1 mm, vias 0 -> 2
- net N$17: track 8.39 -> 83.1 mm, vias 0 -> 1
- net N$44: track 0.00 -> 69.6 mm, vias 0 -> 4
- net N$36: track 0.00 -> 68.0 mm, vias 0 -> 3
- net N$13: track 12.6 -> 76.5 mm, vias 0 -> 2
- net N$15: track 11.3 -> 74.0 mm, vias 0 -> 2
- net N$45: track 0.00 -> 62.5 mm, vias 0 -> 4
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Other:
- board size 87.3 x 81.3 mm -> 52.1 x 66 mm
- board text added: "EnsekiTT"
- board text added: "soraduino"
