File: Soraduino/soraduino.sch (EAGLE design)
At the start: 23 parts, among them IC1 ATMEGA168-AU, IC2 317EMP, IC3 317EMP

Commit message: 回路をとりあえず完成
Parts:
- added R3, R4, R5: 1k, rcl:R-US_R0603
- added RED, YEL1, YEL2: (no value), led:LEDCHIPLED_1206
Connections:
- new net N$10: R3.2, RED.A
- new net N$46: R4.2, YEL1.A
- new net N$48: R5.2, YEL2.A
- net GND: now also RED.C, YEL1.C, YEL2.C
- net N$39: now also R4.1
- net N$40: now also R5.1
- net VCC: now also R3.1
Changed lines of the file:
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@@
 <part name="SUPPLY1" library="supply2" deviceset="GND" device=""/>
 <part name="P+1" library="supply1" deviceset="VCC" device=""/>
+<part name="R3" library="rcl" deviceset="R-US_" device="R0603" value="1k"/>
+<part name="RED" library="led" deviceset="LED" device="CHIPLED_1206"/>
+<part name="YEL1" library="led" deviceset="LED" device="CHIPLED_1206"/>
+<part name="YEL2" library="led" deviceset="LED" device="CHIPLED_1206"/>
+<part name="R4" library="rcl" deviceset="R-US_" device="R0603" value="1k"/>
+<part name="R5" library="rcl" deviceset="R-US_" device="R0603" value="1k"/>
+<part name="FRAME1" library="frames" deviceset="A3L-LOC" device=""/>
 </parts>
 <sheets>
@@
 <instance part="SUPPLY1" gate="GND" x="10.16" y="48.26"/>
 <instance part="P+1" gate="VCC" x="81.28" y="137.16"/>
+<instance part="R3" gate="G$1" x="48.26" y="71.12" rot="R180"/>
+<instance part="RED" gate="G$1" x="40.64" y="71.12" rot="R270"/>
+<instance part="YEL1" gate="G$1" x="264.16" y="2.54"/>
+<instance part="YEL2" gate="G$1" x="259.08" y="2.54"/>
+<instance part="R4" gate="G$1" x="264.16" y="12.7" rot="R270"/>
+<instance part="R5" gate="G$1" x="259.08" y="12.7" rot="R270"/>
+<instance part="FRAME1" gate="G$1" x="-40.64" y="-68.58" smashed="yes">
+<attribute name="DRAWING_NAME" x="303.53" y="-53.34" size="2.54" layer="94" font="vector"/>
+<attribute name="LAST_DATE_TIME" x="303.53" y="-58.42" size="2.286" layer="94" font="vector"/>
+<attribute name="SHEET" x="316.865" y="-63.5" size="2.54" layer="94" font="vector"/>
+</instance>
 </instances>
 <busses>
@@
 <wire x1="208.28" y1="30.48" x2="208.28" y2="25.4" width="0.1524" layer="91"/>
 <wire x1="208.28" y1="25.4" x2="241.3" y2="25.4" width="0.1524" layer="91"/>
+<wire x1="241.3" y1="25.4" x2="264.16" y2="25.4" width="0.1524" layer="91"/>
+<pinref part="R4" gate="G$1" pin="1"/>
+<wire x1="264.16" y1="25.4" x2="264.16" y2="17.78" width="0.1524" layer="91"/>
+<junction x="241.3" y="25.4"/>
 </segment>
 </net>
@@
 <wire x1="205.74" y1="27.94" x2="205.74" y2="22.86" width="0.1524" layer="91"/>
 <wire x1="205.74" y1="22.86" x2="241.3" y2="22.86" width="0.1524" layer="91"/>
+<wire x1="241.3" y1="22.86" x2="259.08" y2="22.86" width="0.1524" layer="91"/>
+<pinref part="R5" gate="G$1" pin="1"/>
+<wire x1="259.08" y1="22.86" x2="259.08" y2="17.78" width="0.1524" layer="91"/>
+<junction x="241.3" y="22.86"/>
 </segment>
 </net>
@@
 <wire x1="17.78" y1="66.04" x2="17.78" y2="50.8" width="0.1524" layer="91"/>
 <wire x1="17.78" y1="50.8" x2="17.78" y2="-2.54" width="0.1524" layer="91"/>
-<wire x1="269.24" y1="-2.54" x2="170.18" y2="-2.54" width="0.1524" layer="91"/>
+<wire x1="269.24" y1="-2.54" x2="264.16" y2="-2.54" width="0.1524" layer="91"/>
+<wire x1="264.16" y1="-2.54" x2="259.08" y2="-2.54" width="0.1524" layer="91"/>
+<wire x1="259.08" y1="-2.54" x2="170.18" y2="-2.54" width="0.1524" layer="91"/>
 <wire x1="170.18" y1="-2.54" x2="160.02" y2="-2.54" width="0.1524" layer="91"/>
 <wire x1="160.02" y1="-2.54" x2="73.66" y2="-2.54" width="0.1524" layer="91"/>
@@
 <wire x1="68.58" y1="81.28" x2="68.58" y2="78.74" width="0.1524" layer="91"/>
 <wire x1="68.58" y1="78.74" x2="68.58" y2="66.04" width="0.1524" layer="91"/>
-<wire x1="68.58" y1="66.04" x2="17.78" y2="66.04" width="0.1524" layer="91"/>
+<wire x1="68.58" y1="66.04" x2="35.56" y2="66.04" width="0.1524" layer="91"/>
 <pinref part="SV2" gate="1" pin="19"/>
 <junction x="68.58" y="124.46"/>
@@
 <junction x="68.58" y="78.74"/>
 <pinref part="JAIRO-ANA" gate="G$1" pin="4"/>
+<wire x1="35.56" y1="66.04" x2="17.78" y2="66.04" width="0.1524" layer="91"/>
 <wire x1="170.18" y1="111.76" x2="172.72" y2="111.76" width="0.1524" layer="91"/>
 <wire x1="243.84" y1="63.5" x2="243.84" y2="48.26" width="0.1524" layer="91"/>
@@
 <pinref part="SUPPLY1" gate="GND" pin="GND"/>
 <junction x="10.16" y="50.8"/>
+<pinref part="RED" gate="G$1" pin="C"/>
+<wire x1="35.56" y1="71.12" x2="35.56" y2="66.04" width="0.1524" layer="91"/>
+<junction x="35.56" y="66.04"/>
+<pinref part="YEL1" gate="G$1" pin="C"/>
+<junction x="264.16" y="-2.54"/>
+<pinref part="YEL2" gate="G$1" pin="C"/>
+<junction x="259.08" y="-2.54"/>
 </segment>
 </net>
@@
 <wire x1="81.28" y1="134.62" x2="81.28" y2="127" width="0.1524" layer="91"/>
 <junction x="81.28" y="127"/>
+<pinref part="R3" gate="G$1" pin="1"/>
+<wire x1="71.12" y1="71.12" x2="53.34" y2="71.12" width="0.1524" layer="91"/>
+<junction x="71.12" y="71.12"/>
 </segment>
 </net>
@@
 </segment>
 </net>
+<net name="N$10" class="0">
+<segment>
+<pinref part="R3" gate="G$1" pin="2"/>
+<pinref part="RED" gate="G$1" pin="A"/>
+</segment>
+</net>
+<net name="N$46" class="0">
+<segment>
+<pinref part="R4" gate="G$1" pin="2"/>
+<pinref part="YEL1" gate="G$1" pin="A"/>
+<wire x1="264.16" y1="5.08" x2="264.16" y2="7.62" width="0.1524" layer="91"/>
+</segment>
+</net>
+<net name="N$48" class="0">
+<segment>
+<pinref part="R5" gate="G$1" pin="2"/>
+<pinref part="YEL2" gate="G$1" pin="A"/>
+<wire x1="259.08" y1="5.08" x2="259.08" y2="7.62" width="0.1524" layer="91"/>
+</segment>
+</net>
